File: Senior Project/Fuel_Injection/schematic.sch (EAGLE design)
At the start: 6 parts, among them IC1 7805T

Commit message: Add files via upload
Parts:
- removed SPARK_PLUG: (no value), con-molex:KK-156-4
- added C1: (no value), rcl:CPOL-USE2.5-5
- added C2: 0.33uf, rcl:CPOL-USE2.5-5
- added C3: 0.1uf, rcl:CPOL-USE2.5-5
- added POWER_N_MOSFET2, POWER_N_MOSFET3: 30N06L, transistor-power:IRF520
- added SPARK_PLUG_GND, SPARK_PLUG_POWER: (no value), con-molex:KK-156-2
- added X2: TSW-140-07-G-S, con-samtec:TSW-140-07-G-S
- R1: value (none) -> 10K
- renumbered POWER_MOSFET to POWER_N_MOSFET
Connections:
- new net 0: C2.-, C3.-, IC1.GND, POWER_N_MOSFET2.S, POWER_N_MOSFET3.S
- new net N$1: POWER_N_MOSFET3.G, X2-1.1
- new net N$2: POWER_N_MOSFET2.G, X2-2.1
- new net N$3: POWER_N_MOSFET3.D, SPARK_PLUG_GND-1.S
- new net N$4: POWER_N_MOSFET2.D, SPARK_PLUG_GND-2.S
- new net VCC: C2.+, C3.+, IC1.VI, IC1.VO, SPARK_PLUG_POWER-1.S, SPARK_PLUG_POWER-2.S
Other:
- moved on the sheet: IC1

Commit message: Add files via upload
Parts:
- removed C1: (no value), rcl:CPOL-USE2.5-5
- removed POWER_N_MOSFET: 30N06L, transistor-power:IRF520
- added CRANK_SENSOR: (no value), con-molex:KK-156-2
- added R2, R3, R4: 10K, rcl:R-US_0207/7
Connections:
- new net N$5: LEVEL_SHIFTER.S, R1.1, X2-3.1
- new net N$6: LEVEL_SHIFTER.G, R1.2
- new net N$7: CRANK_SENSOR-1.S, LEVEL_SHIFTER.D, R2.1
- net 0: now also R3.2, R4.2
- net N$1: now also R4.1
- net N$2: now also R3.1
- net VCC: now also R2.2
Other:
- moved on the sheet: FUEL_INJECTOR-1, FUEL_INJECTOR-2, FUEL_INJECTOR-3, FUEL_INJECTOR-4, LEVEL_SHIFTER, R1, X2-3
